Commit message: HOST for ths_23dof

File: legged_gym/resources/robots/ths_23dof/urdf/ths_23dof.urdf (robot description, URDF)
Before this commit: robot ths_23dof, 31 links, 30 joints
Joints:
- joint left_hip_pitch_joint: limit lower=-2 upper=2 effort=88 velocity=10 -> lower=-2.0 upper=2 effort=88 velocity=10
